Commit message: water pouring with 3D mouse

File: specification/urdf/objects/glass1.urdf (robot description, URDF)
Before this commit: robot glass1, 1 links, 0 joints
Links:
- link root: geometry collision mesh filename=../../meshes/objects/glass1_vhacd.obj scale=0.04 0.04 0.04; visual mesh filename=../../meshes/objects/glass1.obj scale=0.04 0.04 0.04
