Commit message: pen kitting simulator works

File: specification/urdf/objects/pen_cavity.urdf (robot description, URDF)
Before this commit: robot pen_cavity, 3 links, 2 joints
Links:
- link pen_cavity_out: geometry collision mesh filename=../../meshes/objects/pen_cavity_in_out.obj scale=0.001 0.001 0.001; visual mesh filename=../../meshes/objects/pen_cavity_out.obj scale=0.001 0.001 0.001

File: specification/urdf/robots/arm_and_gripper.urdf.xacro (robot description, xacro)
@@ -24,30 +24,30 @@
     <origin xyz="0 0 0" rpy="0 0 0"/>
   </xacro:robotiq_85_gripper>
-  <link name="peg">
-    <inertial>
-      <origin rpy="0 0 0" xyz="0 0 0.24"/>
-      <mass value="0.4"/>
-      <inertia ixx="0.0094" ixy="0" ixz="0" iyy="0.0008" iyz="0" izz="0.0094"/>
-    </inertial>
-    <visual>
-      <origin rpy="0, 1.57, 0" xyz="0.12, 0, 0"/>
-      <geometry>
-	<mesh filename="../../meshes/objects/peg.obj" scale="0.001 0.001 0.001"/>
-      </geometry>
-      <material name="blue">
-        <color rgba="0.5 0.5 1.0 1"/>
-      </material>
-    </visual>
-    <collision>
-      <origin rpy="0, 1.57, 0" xyz="0.12, 0, 0"/>
-      <geometry>
-	<mesh filename="../../meshes/objects/peg.obj" scale="0.001 0.001 0.001"/>
-      </geometry>
-    </collision>
-  </link>
-  <joint name="hand_to_peg" type="fixed">
-    <parent link="c_bot_gripper_coupling_flange_link"/>
-    <child link="peg"/>
-    <axis xyz="0 0 1"/>
-  </joint>
+  <!-- <link name="peg"> -->
+  <!--   <inertial> -->
+  <!--     <origin rpy="0 0 0" xyz="0 0 0.24"/> -->
+  <!--     <mass value="0.4"/> -->
+  <!--     <inertia ixx="0.0094" ixy="0" ixz="0" iyy="0.0008" iyz="0" izz="0.0094"/> -->
+  <!--   </inertial> -->
+  <!--   <visual> -->
+  <!--     <origin rpy="0, 1.57, 0" xyz="0.12, 0, 0"/> -->
+  <!--     <geometry> -->
+  <!--       <mesh filename="../../meshes/objects/peg.obj" scale="0.001 0.001 0.001"/> -->
+  <!--     </geometry> -->
+  <!--     <material name="blue"> -->
+  <!--       <color rgba="0.5 0.5 1.0 1"/> -->
+  <!--     </material> -->
+  <!--   </visual> -->
+  <!--   <collision> -->
+  <!--     <origin rpy="0, 1.57, 0" xyz="0.12, 0, 0"/> -->
+  <!--     <geometry> -->
+  <!--       <mesh filename="../../meshes/objects/peg.obj" scale="0.001 0.001 0.001"/> -->
+  <!--     </geometry> -->
+  <!--   </collision> -->
+  <!-- </link> -->
+  <!-- <joint name="hand_to_peg" type="fixed"> -->
+  <!--   <parent link="c_bot_gripper_coupling_flange_link"/> -->
+  <!--   <child link="peg"/> -->
+  <!--   <axis xyz="0 0 1"/> -->
+  <!-- </joint> -->
 </robot>
