Commit message: peg-in-hole task

File: specification/urdf/objects/large_table.urdf (robot description, URDF)
Before this commit: robot cabinet, 2 links, 1 joints
Links:
- link link_ext: geometry collision box size=1.6 1.6 0.005; visual box size=1.6 1.6 0.01

Commit message: random placing and force estimation

File: specification/urdf/objects/large_table.urdf (robot description, URDF)
Before this commit: robot cabinet, 2 links, 1 joints
Links:
- removed link link_cab
- removed link link_ext
- added link table_top; collision box size=1.6 1.6 0.01; visual box size=1.6 1.6 0.01
Joints:
- removed joint joint_cabExt

Commit message: flake8 compliance

File: specification/urdf/objects/large_table.urdf (robot description, URDF)
Before this commit: robot table, 1 links, 0 joints
Links:
- link table_top: mass None -> .0
