Commit message: adding procedual teaching

File: specification/urdf/arm_and_gripper/ur5e_pen.urdf.xacro (robot description, xacro)
@@ -34,5 +34,5 @@
     </inertial>
     <visual>
-      <origin rpy="0 -1.0 0" xyz="0.18 0 0.05"/>
+      <origin rpy="0 -1.0 0" xyz="0.19 0 0.05"/>
       <material name="pen_color"/>
       <geometry>
@@ -41,5 +41,5 @@
     </visual>
     <collision>
-      <origin rpy="0 -1.0 0" xyz="0.18 0 0.05"/>
+      <origin rpy="0 -1.0 0" xyz="0.19 0 0.05"/>
       <geometry>
         <mesh filename="../../meshes/objects/pen_vhacd.obj" scale="0.001 0.001 0.001"/>
